File: face_plate/wvtbl_face_plate.kicad_pcb (KiCad board)
At the start: 2 copper layers, 30 x 128.5 mm, 10 parts, among them U1 WVTBL

Commit message: Main board PCB
Other:
- board text added: "JLCJLCJLCJLC"
Changed lines of the file:
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@@
   (gr_line (start 42.5 109) (end 42.5 78.5) (layer "F.SilkS") (width 0.6))
   (gr_line (start 57.5 98.5) (end 57.5 109) (layer "F.SilkS") (width 0.6))
+  (gr_text "JLCJLCJLCJLC" (at 50 45) (layer "B.SilkS")
+    (effects (font (size 1 1) (thickness 0.15)) (justify mirror))
+  )
   (zone (net 1) (net_name "GND") (layer "F.Cu") (hatch edge 0.508)
     (connect_pads yes (clearance 0))
