File: face_plate/wvtbl_face_plate.kicad_sch (KiCad schematic)
At the start: 10 parts, among them U1 WVTBL

Commit message: Corrections on faceplate holes place and sizes
Parts:
- H101: footprint WITNS:PotentiometerHole_7.4mm_M7_Pad -> WITNS:EncoderHole_9.4mm_M9_Pad
Changed lines of the file:
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@@
       (effects (font (size 1.27 1.27)) (justify left))
     )
-    (property "Footprint" "WITNS:PotentiometerHole_7.4mm_M7_Pad" (id 2) (at 69.85 44.45 0)
+    (property "Footprint" "WITNS:EncoderHole_9.4mm_M9_Pad" (id 2) (at 69.85 44.45 0)
       (effects (font (size 1.27 1.27)) hide)
     )
@@
     )
     (path "/1627844d-d79a-4682-a0c6-a6ffcdb8ff06"
-      (reference "H101") (unit 1) (value "Pitch") (footprint "WITNS:PotentiometerHole_7.4mm_M7_Pad")
+      (reference "H101") (unit 1) (value "Pitch") (footprint "WITNS:EncoderHole_9.4mm_M9_Pad")
     )
     (path "/26c86062-2af5-48eb-9445-359a8c5d590b"
