File: processing_board/stm32.kicad_sch (KiCad schematic)
At the start: 19 parts, among them J7 Conn_02x07_Odd_Even, SW201 RST, U201 STM32G431KBT6, Y201 16MHz

Commit message: Main board PCB
Other:
- note added: "5V tolerant"
Changed lines of the file:
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@@
+    (stroke (width 0) (type default) (color 0 0 0 0))
+  )
+  (polyline (pts (xy 247.65 97.79) (xy 250.19 97.79))
     (stroke (width 0) (type default) (color 0 0 0 0))
   )
@@
     (stroke (width 0) (type default) (color 0 0 0 0))
   )
+  (polyline (pts (xy 247.65 92.71) (xy 250.19 92.71))
+    (stroke (width 0) (type default) (color 0 0 0 0))
+  )
+  (polyline (pts (xy 250.19 92.71) (xy 250.19 97.79))
+    (stroke (width 0) (type default) (color 0 0 0 0))
+  )
   (wire (pts (xy 233.68 34.29) (xy 233.68 35.56))
     (stroke (width 0) (type default) (color 0 0 0 0))
@@
     (stroke (width 0) (type default) (color 0 0 0 0))
   )
+  (text "5V tolerant" (at 251.46 93.98 0)
+    (effects (font (size 1.27 1.27)) (justify left bottom))
+  )
   (text "Bypass capacitors\n100nF as close to STM32 VDD as possible\n4.7uF just next to the 100nF"
