File: processing_board/witns_processing_board.kicad_pcb (KiCad board)
At the start: 4 copper layers, 29 x 45 mm, 63 parts, among them J101 Conn_01x13, J102 Conn_01x05, J103 Conn_01x09, J7 Conn_02x07_Odd_Even, SW201 RST, U201 STM32G431KBT6, U301 MCP6002-E/SN, U302 MCP6002-E/SN, U303 TL072CDR, U401 BU33SD5WG-TR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

Commit message: Main board PCB
Connections:
- J101 pad 6: GND -> +3.3VA
- J103 pad 1: GND -> +3V3
Other:
- board text added: "JLCJLCJLCJLC"
Changed lines of the file:
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@@
     (fp_line (start 1.27 1.27) (end 1.27 -21.59) (layer "B.Fab") (width 0.1))
     (pad "1" thru_hole rect (at 0 0 180) (size 1.7 1.7) (drill 1) (layers *.Cu *.Mask)
-      (net 1 "GND") (pinfunction "Pin_1") (pintype "passive"))
+      (net 2 "+3V3") (pinfunction "Pin_1") (pintype "passive"))
     (pad "2" thru_hole oval (at 0 -2.54 180) (size 1.7 1.7) (drill 1) (layers *.Cu *.Mask)
       (net 27 "/STM32/ENCODER_SWITCH") (pinfunction "Pin_2") (pintype "passive"))
@@
       (net 8 "/POT_4") (pinfunction "Pin_5") (pintype "passive"))
     (pad "6" thru_hole oval (at 0 -12.7 180) (size 1.7 1.7) (drill 1) (layers *.Cu *.Mask)
-      (net 1 "GND") (pinfunction "Pin_6") (pintype "passive"))
+      (net 3 "+3.3VA") (pinfunction "Pin_6") (pintype "passive"))
     (pad "7" thru_hole oval (at 0 -15.24 180) (size 1.7 1.7) (drill 1) (layers *.Cu *.Mask)
       (net 17 "/Analog Front-end/RACK_CV1") (pinfunction "Pin_7") (pintype "passive"))
@@
     )
   )
+  (gr_circle (center 47.6 105.2) (end 47.711803 105.2) (layer "F.SilkS") (width 0.3) (fill none))
   (gr_line (start 57 101) (end 59 101) (layer "F.SilkS") (width 0.15))
   (gr_line (start 59.5 104.5) (end 59.5 103.5) (layer "F.SilkS") (width 0.15))
@@
     (effects (font (size 1 1) (thickness 0.15)) (justify left mirror))
   )
+  (gr_text "JLCJLCJLCJLC" (at 52.5 94.5) (layer "B.SilkS")
+    (effects (font (size 1 1) (thickness 0.15)) (justify mirror))
+  )
   (gr_text "EncB" (at 61.43 107.62) (layer "B.SilkS")
