File: processing_board/witns_processing_board.kicad_sch (KiCad schematic)
At the start: 3 parts, among them J101 Conn_01x13, J102 Conn_01x05, J103 Conn_01x09

Commit message: Main board PCB
Connections:
- net GND: no longer J101.6 (Pin_6), J103.1 (Pin_1)
- new net +3.3VA: J101.6 (Pin_6)
- new net +3V3: J103.1 (Pin_1)
Changed lines of the file:
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@@
   (junction (at 115.57 110.49) (diameter 0) (color 0 0 0 0)
   )
-  (junction (at 69.85 67.31) (diameter 0) (color 0 0 0 0)
-  )
-  (junction (at 115.57 100.33) (diameter 0) (color 0 0 0 0)
-  )
-  (junction (at 69.85 62.23) (diameter 0) (color 0 0 0 0)
-  )
-  (junction (at 69.85 49.53) (diameter 0) (color 0 0 0 0)
+  (junction (at 73.66 67.31) (diameter 0) (color 0 0 0 0)
+  )
+  (junction (at 73.66 62.23) (diameter 0) (color 0 0 0 0)
   )
   (junction (at 64.77 176.53) (diameter 0) (color 0 0 0 0)
@@
     (stroke (width 0) (type default) (color 0 0 0 0))
   )
-  (wire (pts (xy 69.85 67.31) (xy 69.85 68.58))
+  (wire (pts (xy 73.66 67.31) (xy 73.66 68.58))
     (stroke (width 0) (type default) (color 0 0 0 0))
   )
@@
     (stroke (width 0) (type default) (color 0 0 0 0))
   )
-  (wire (pts (xy 62.23 49.53) (xy 69.85 49.53))
-    (stroke (width 0) (type default) (color 0 0 0 0))
-  )
   (wire (pts (xy 114.3 105.41) (xy 157.48 105.41))
     (stroke (width 0) (type default) (color 0 0 0 0))
   )
-  (wire (pts (xy 115.57 90.17) (xy 115.57 100.33))
-    (stroke (width 0) (type default) (color 0 0 0 0))
-  )
   (wire (pts (xy 52.07 171.45) (xy 64.77 171.45))
     (stroke (width 0) (type default) (color 0 0 0 0))
@@
     (stroke (width 0) (type default) (color 0 0 0 0))
   )
-  (wire (pts (xy 69.85 49.53) (xy 69.85 36.83))
-    (stroke (width 0) (type default) (color 0 0 0 0))
-  )
   (wire (pts (xy 154.94 77.47) (xy 157.48 77.47))
     (stroke (width 0) (type default) (color 0 0 0 0))
@@
     (stroke (width 0) (type default) (color 0 0 0 0))
   )
-  (wire (pts (xy 114.3 90.17) (xy 115.57 90.17))
-    (stroke (width 0) (type default) (color 0 0 0 0))
-  )
-  (wire (pts (xy 62.23 67.31) (xy 69.85 67.31))
+  (wire (pts (xy 62.23 67.31) (xy 73.66 67.31))
     (stroke (width 0) (type default) (color 0 0 0 0))
   )
@@
     (stroke (width 0) (type default) (color 0 0 0 0))
   )
-  (wire (pts (xy 69.85 67.31) (xy 69.85 62.23))
-    (stroke (width 0) (type default) (color 0 0 0 0))
-  )
-  (wire (pts (xy 69.85 62.23) (xy 69.85 49.53))
+  (wire (pts (xy 73.66 67.31) (xy 73.66 62.23))
+    (stroke (width 0) (type default) (color 0 0 0 0))
+  )
+  (wire (pts (xy 73.66 36.83) (xy 73.66 62.23))
     (stroke (width 0) (type default) (color 0 0 0 0))
   )
@@
     (stroke (width 0) (type default) (color 0 0 0 0))
   )
+  (wire (pts (xy 118.11 88.9) (xy 118.11 90.17))
+    (stroke (width 0) (type default) (color 0 0 0 0))
+  )
   (wire (pts (xy 62.23 54.61) (xy 101.6 54.61))
     (stroke (width 0) (type default) (color 0 0 0 0))
   )
+  (wire (pts (xy 118.11 90.17) (xy 114.3 90.17))
+    (stroke (width 0) (type default) (color 0 0 0 0))
+  )
   (wire (pts (xy 115.57 100.33) (xy 115.57 110.49))
     (stroke (width 0) (type default) (color 0 0 0 0))
@@
     (stroke (width 0) (type default) (color 0 0 0 0))
   )
-  (wire (pts (xy 69.85 36.83) (xy 62.23 36.83))
+  (wire (pts (xy 73.66 36.83) (xy 62.23 36.83))
     (stroke (width 0) (type default) (color 0 0 0 0))
   )
@@
     (stroke (width 0) (type default) (color 0 0 0 0))
   )
-  (wire (pts (xy 62.23 62.23) (xy 69.85 62.23))
+  (wire (pts (xy 62.23 62.23) (xy 73.66 62.23))
     (stroke (width 0) (type default) (color 0 0 0 0))
   )
@@
     (pin "9")
   )
+  (symbol (lib_id "power:+3.3V") (at 118.11 88.9 0) (unit 1)
+    (in_bom yes) (on_board yes)
+    (property "Reference" "#PWR0114" (id 0) (at 118.11 92.71 0)
+      (effects (font (size 1.27 1.27)) hide)
+    )
+    (property "Value" "+3.3V" (id 1) (at 118.11 85.09 0))
+    (property "Footprint" "" (id 2) (at 118.11 88.9 0)
+      (effects (font (size 1.27 1.27)) hide)
+    )
+    (property "Datasheet" "" (id 3) (at 118.11 88.9 0)
+      (effects (font (size 1.27 1.27)) hide)
+    )
+    (pin "1")
+  )
   (symbol (lib_id "Connector_Generic:Conn_01x05") (at 46.99 173.99 0) (mirror y) (unit 1)
     (in_bom yes) (on_board yes) (fields_autoplaced)
@@
     (pin "1")
   )
-  (symbol (lib_id "power:GND") (at 69.85 68.58 0) (unit 1)
-    (in_bom yes) (on_board yes) (fields_autoplaced)
-    (property "Reference" "#PWR0101" (id 0) (at 69.85 74.93 0)
-      (effects (font (size 1.27 1.27)) hide)
-    )
-    (property "Value" "GND" (id 1) (at 69.85 73.66 0))
-    (property "Footprint" "" (id 2) (at 69.85 68.58 0)
-      (effects (font (size 1.27 1.27)) hide)
-    )
-    (property "Datasheet" "" (id 3) (at 69.85 68.58 0)
+  (symbol (lib_id "power:+3.3VA") (at 62.23 49.53 270) (mirror x) (unit 1)
+    (in_bom yes) (on_board yes)
+    (property "Reference" "#PWR?" (id 0) (at 58.42 49.53 0)
+      (effects (font (size 1.27 1.27)) hide)
+    )
+    (property "Value" "+3.3VA" (id 1) (at 68.58 49.53 90))
+    (property "Footprint" "" (id 2) (at 62.23 49.53 0)
+      (effects (font (size 1.27 1.27)) hide)
+    )
+    (property "Datasheet" "" (id 3) (at 62.23 49.53 0)
+      (effects (font (size 1.27 1.27)) hide)
+    )
+    (pin "1")
+  )
+  (symbol (lib_id "power:GND") (at 73.66 68.58 0) (unit 1)
+    (in_bom yes) (on_board yes) (fields_autoplaced)
+    (property "Reference" "#PWR0101" (id 0) (at 73.66 74.93 0)
+      (effects (font (size 1.27 1.27)) hide)
+    )
+    (property "Value" "GND" (id 1) (at 73.66 73.66 0))
+    (property "Footprint" "" (id 2) (at 73.66 68.58 0)
+      (effects (font (size 1.27 1.27)) hide)
+    )
+    (property "Datasheet" "" (id 3) (at 73.66 68.58 0)
       (effects (font (size 1.27 1.27)) hide)
     )
@@
       (reference "#PWR0113") (unit 1) (value "+3.3VA") (footprint "")
     )
+    (path "/4b8a7d9a-3fe1-4b65-bd62-fdd7fcfdce9b"
+      (reference "#PWR0114") (unit 1) (value "+3.3V") (footprint "")
+    )
     (path "/ae2e9975-cb8b-4be5-ade8-02890e89b212/50ba2ba6-03a9-4c65-9479-19f1bbdb98e2"
       (reference "#PWR0201") (unit 1) (value "GND") (footprint "")
@@
       (reference "#PWR0404") (unit 1) (value "GND") (footprint "")
     )
+    (path "/958ea753-3982-4aba-aa1d-5ee89b48a571"
+      (reference "#PWR?") (unit 1) (value "+3.3VA") (footprint "")
+    )
     (path "/ae2e9975-cb8b-4be5-ade8-02890e89b212/33ea93d2-f72e-4a83-8cbc-f5e9c6711234"
